Commit message: modified simulation

File: simulation_ws/install/yahboomcar_description/share/yahboomcar_description/urdf/MicroROS.urdf (robot description, URDF)
Before this commit: robot micro4.0, 9 links, 8 joints
Joints:
- joint radar_Joint: origin xyz=0 0 0.078933557468359 rpy=0 0 0 -> xyz=0 0.02 0.078933557468359 rpy=0 0 0
